Commit message: correct some runtime errors, errors still exist, for more details, please read record.md

File: ocs2_dancer/dancer_description/urdf/dancer.urdf (robot description, URDF)
Before this commit: robot human, 19 links, 18 joints
Links:
- added link left_shoulder, mass 0.044031000000000001; visual mesh filename=package://dancer_description/urdf/meshes/left_shoulder.STL scale=1 1 1
- added link right_shoulder, mass 0.051527000000000003; visual mesh filename=package://dancer_description/urdf/meshes/right_shoulder.STL scale=1 1 1
- link chest: mass 0.88192504598295396 -> 0.18192504598295396; geometry collision box size=0.1125 0.0975 0.14; collision cylinder length=0.1146 radius=0.008
- link head: geometry collision sphere radius=0.0284086; collision sphere radius=0.0305397
- link left_arm: mass 0.140880482426088 -> 0.14643999999999999; geometry visual mesh filename=package://dancer_description/urdf/meshes/left_arm.STL scale=1 1 1
- link left_foot: geometry collision box size=0.0659544 0.149954 0.012; collision box size=0.087 0.147 0.006
- link left_hand: mass 0.024044269196268502 -> 0.064269999999999994; geometry visual mesh filename=package://dancer_description/urdf/meshes/left_hand.STL scale=1 1 1
- link left_leg_ankle: geometry collision box size=0.003 0.029 0.0651; collision box size=0.0035 0.029 0.0651
- link left_leg_knee: geometry collision cylinder length=0.0055 radius=0.014; collision cylinder length=0.0055 radius=0.014
- link left_leg_pitch: geometry collision box size=0.0539 0.0402 0.0015; collision box size=0.0539 0.0402 0.0015
- link left_leg_roll: geometry collision box size=0.028997 0.0035 0.0553928; collision box size=0.0403884 0.038 0.0611006
- link left_leg_yaw: geometry collision box size=0.041 0.0637 0.003; visual mesh filename=package://dancer_description/urdf/meshes/left_leg_yaw.STL scale=1 1 1
- link neck: geometry collision box size=0.0302 0.0356 0.0396; collision box size=0.0342 0.0355 0.015
- link right_arm: mass 0.140880482426088 -> 0.13894999999999999; geometry visual mesh filename=package://dancer_description/urdf/meshes/right_arm.STL scale=1 1 1
- link right_foot: geometry collision box size=0.0659544 0.149954 0.012; collision box size=0.087 0.147 0.006
- link right_hand: mass 0.024044269196268502 -> 0.064269999999999994; geometry visual mesh filename=package://dancer_description/urdf/meshes/right_hand.STL scale=1 1 1
- link right_leg_ankle: geometry collision box size=0.003 0.029 0.0651; collision box size=0.0035 0.029 0.0651
- link right_leg_knee: geometry collision cylinder length=0.0055 radius=0.014; collision cylinder length=0.0055 radius=0.014
- link right_leg_pitch: geometry collision box size=0.0539 0.0402 0.0015; collision box size=0.0539 0.0402 0.0015
- link right_leg_roll: geometry collision box size=0.028997 0.0035 0.0553928; collision box size=0.0403884 0.038 0.0611006
- link right_leg_yaw: geometry collision box size=0.041 0.0637 0.003; visual mesh filename=package://dancer_description/urdf/meshes/right_leg_yaw.STL scale=1 1 1
Joints:
- added joint left_arm_middle: type revolute, parent left_shoulder, child left_arm, origin xyz=0.028100000000000007 0.025800000000000003 -0.029 rpy=0.0 0.0 0.0, axis -1 0 0, limit lower=0 upper=0 effort=0 velocity=0
- added joint right_arm_middle: type revolute, parent right_shoulder, child right_arm, origin xyz=-0.022 -0.028999999999999998 -0.029 rpy=0.0 0.0 0.0, axis 1 0 0, limit lower=0 upper=0 effort=0 velocity=0
- joint head_pitch: limit lower=-3.141592654 upper=3.141592654 effort=3 velocity=20 -> lower=-3.14159265359 upper=3.14159265359 effort=3 velocity=20; origin xyz=-0.018750 0.000000 0.043800  rpy=1.570796 -1.491213 -1.570796  -> xyz=-0.0187500000000007 -3.469446951953614e-18 0.04379999999999995 rpy=1.5707963267948957 -1.4912133887083963 -1.570796326794886; type fixed -> revolute
- joint head_yaw: limit lower=-3.141592654 upper=3.141592654 effort=3 velocity=20 -> lower=-3.14159265359 upper=3.14159265359 effort=3 velocity=20; origin xyz=0 0.0134 0.020750000000000046 rpy=0.000000 0.000000 0.000000  -> xyz=0.0 0.0134 0.020750000000000046 rpy=0.0 0.0 0.0; type fixed -> revolute
- joint left_ankle_pitch: limit lower=-3.141592654 upper=3.141592654 effort=10 velocity=20 -> lower=-3.14159265359 upper=3.14159265359 effort=10 velocity=20; origin xyz=0.129998462179975 -0.000211229839968 0.000595997311238  rpy=2.96537 1.58011 -0.174599  -> xyz=0.12999999999999534 1.214306433183765e-17 -4.579669976578771e-16 rpy=3.14159265358979 1.5707963267948952 0.0
- joint left_ankle_roll: limit lower=-3.141592654 upper=3.141592654 effort=7 velocity=20 -> lower=-3.14159265359 upper=3.14159265359 effort=3 velocity=20; origin xyz=0.023387 -0.069538 -0.000113445  rpy=0.0 0.0 0.0  -> xyz=0.02349999999999914 -0.0694999999999985 -1.1102230246251565e-15 rpy=-6.3439431139357456e-18 -0.0045846107623825905 3.943480964427586e-18
- joint left_arm_lower: axis 0 0 -1 -> 0 -1 0; limit lower=-3.141592654 upper=3.141592654 effort=3 velocity=20 -> lower=-3.0 upper=3.0 effort=3 velocity=20; origin xyz=0.136000 0 0.04955 rpy=0.0 0.0 0.0  -> xyz=-0.028100000000000003 0.023349999999999982 -0.1076 rpy=0.0 1.5700000000000003 0.0
- joint left_arm_upper: axis 0 0 -1 -> 0 -1 0; child left_arm -> left_shoulder; limit lower=-3.141592654 upper=3.141592654 effort=7 velocity=20 -> lower=-3.14159265359 upper=3.14159265359 effort=3 velocity=20; origin xyz=-0.074700 0.013400 0.000000  rpy=3.141593 1.570796 0.000000  -> xyz=-0.077 0.0134 0.0 rpy=0.0 0.0 1.5707963267948963
- joint left_hip_pitch: limit lower=-3.141592654 upper=3.141592654 effort=10 velocity=20 -> lower=-3.14159265359 upper=3.14159265359 effort=10 velocity=20; origin xyz=-0.028999695 0.0292 0.000132953  rpy=-0.340598 1.565932 2.800991  -> xyz=-0.028999695229219802 0.0292000000000009 0.00013295342185881687 rpy=-0.34059803684003587 1.5659322938814761 2.80099089209511
- joint left_hip_roll: limit lower=-3.141592654 upper=3.141592654 effort=7 velocity=20 -> lower=-3.14159265359 upper=3.14159265359 effort=3 velocity=20; origin xyz=0.0 -0.0292 -0.055  rpy=0.000000 0.000000 0.000000  -> xyz=0.0 -0.0291999999999996 -0.055000000000000104 rpy=0.0 0.0 0.0
- joint left_hip_yaw: limit lower=-3.141592654 upper=3.141592654 effort=7 velocity=20 -> lower=-3.14159265359 upper=3.14159265359 effort=3 velocity=20; origin xyz=-0.044999999999999998 0.0133599999999985 -0.16994999999999999  rpy=0.000000 0.000000 0.000000  -> xyz=-0.045 0.0133599999999985 -0.16995 rpy=0.0 0.0 0.0
- joint left_knee: limit lower=-3.141592654 upper=3.141592654 effort=10 velocity=20 -> lower=-3.14159265359 upper=3.14159265359 effort=10 velocity=20; origin xyz=0.130023677484126 -0.000211229839968 -0.004903944887406  rpy=0 0 0  -> xyz=0.12999999999999962 1.0113437864944785e-15 -0.00550000000000285 rpy=3.3406840085472114e-16 2.1316282072803006e-14 7.672907131907189e-15
- joint right_ankle_pitch: limit lower=-3.141592654 upper=3.141592654 effort=10 velocity=20 -> lower=-3.14159265359 upper=3.14159265359 effort=10 velocity=20; origin xyz=0.129976266544291 0.000489901482115 0.003942097378979  rpy=1.56716 -1.56838 -1.57091  -> xyz=0.13000000000000012 2.5240226575462543e-15 0.003100000000003933 rpy=-0.0013797295538484633 -1.5707963267948617 0.0
- joint right_ankle_roll: limit lower=-3.141592654 upper=3.141592654 effort=7 velocity=20 -> lower=-3.14159265359 upper=3.14159265359 effort=3 velocity=20; origin xyz=-0.0267659  -0.0694361 -0.000164943 rpy=3.1392 3.13511 3.14158  -> xyz=-0.026600000000000082 -0.06950000000000016 1.6653345369377348e-16 rpy=-8.189825335909092e-19 0.0 -1.3596032129378206e-18
- joint right_arm_lower: axis 0 0 1 -> 0 -1 0; limit lower=-3.141592654 upper=3.141592654 effort=3 velocity=20 -> lower=-3.0 upper=3.0 effort=3 velocity=20; origin xyz=0.136000 0 0.05255  rpy=0.000000 0.0 0.000000  -> xyz=0.022 0.019250000000000003 -0.1076 rpy=0.0 1.5700000000000003 0.0
- joint right_arm_upper: axis 0 0 1 -> 0 -1 0; child right_arm -> right_shoulder; limit lower=-3.141592654 upper=3.141592654 effort=7 velocity=20 -> lower=-3.14159265359 upper=3.14159265359 effort=3 velocity=20; origin xyz=0.074700 0.013400 0.000000  rpy=0.000000 1.570796 0.000000  -> xyz=0.0747 0.0134 0.0 rpy=0.0 0.0 1.5707963267948963
- joint right_hip_pitch: limit lower=-3.141592654 upper=3.141592654 effort=10 velocity=20 -> lower=-3.14159265359 upper=3.14159265359 effort=10 velocity=20; origin xyz=0.029 0.0292 0  rpy=1.57078 1.56703  1.5708  -> xyz=0.028999999999999304 0.0292 2.7755575615628914e-17 rpy=1.5707963267974303 1.56702784493591 1.5707963267974459
- joint right_hip_roll: axis 0 -1 0 -> 0 1 0; limit lower=-3.141592654 upper=3.141592654 effort=7 velocity=20 -> lower=-3.14159265359 upper=3.14159265359 effort=3 velocity=20; origin xyz=0.0 -0.0292 -0.055  rpy=0.000000 -0.006478 0.000000  -> xyz=0.0 -0.0291999999999996 -0.055000000000000104 rpy=0.0 -0.006478263843886278 0.0
- joint right_hip_yaw: axis 0 0 -1 -> 0 0 1; limit lower=-3.141592654 upper=3.141592654 effort=7 velocity=20 -> lower=-3.14159265359 upper=3.14159265359 effort=3 velocity=20; origin xyz=0.045000 0.013360 -0.169950  rpy=0.000000 0.000000 0.000000  -> xyz=0.045 0.0133599999999985 -0.16995 rpy=0.0 0.0 0.0
- joint right_knee: limit lower=-3.141592654 upper=3.141592654 effort=10 velocity=20 -> lower=-3.14159265359 upper=3.14159265359 effort=10 velocity=20; origin xyz=0.130031979223655 0.000489901482115 -0.004657722159670  rpy=0.0 0.0 0.0  -> xyz=0.13000000000000006 6.314393452555578e-16 -0.005499999999998409 rpy=8.26353924749796e-16 2.6201263381153694e-14 -1.4487316805982308e-14

Commit message: modify urdf file, change some joint type from revolute to fixed

File: ocs2_dancer/dancer_description/urdf/dancer.urdf (robot description, URDF)
Before this commit: robot robot, 21 links, 20 joints
Joints:
- joint head_pitch: type revolute -> fixed
- joint head_yaw: type revolute -> fixed
- joint left_arm_lower: type revolute -> fixed
- joint left_arm_middle: type revolute -> fixed
- joint left_arm_upper: type revolute -> fixed
- joint right_arm_lower: type revolute -> fixed
- joint right_arm_middle: type revolute -> fixed
- joint right_arm_upper: type revolute -> fixed

Commit message: modify dancer_controllers package add somm cpp files and a launch file. For more details, please read record.md

File: ocs2_dancer/dancer_description/urdf/dancer.urdf (robot description, URDF)
Before this commit: robot robot, 21 links, 20 joints
Links:
- added link virtual, mass 0.0
Joints:
- added joint chest_to_virtual: type fixed, parent virtual, child chest, origin xyz=0 0 0 rpy=0 0 -1.570796327
- joint left_arm_upper: origin xyz=-0.077 0.0134 0.0 rpy=0.0 0.0 1.5707963267948963 -> xyz=-0.077 0.0134 0.0 rpy=0.0 0.0 1.570796327
- joint right_arm_upper: origin xyz=0.0747 0.0134 0.0 rpy=0.0 0.0 1.5707963267948963 -> xyz=0.0747 0.0134 0.0 rpy=0.0 0.0 1.570796327
